Commit message: Adding Water & Soap Tank on Mobile Base

File: src/my_robot_description/urdf/common_properties.xacro (robot description, xacro)
@@ -12,4 +12,7 @@
         <material name="yellow">
             <color rgba="1 1 0 1"/>
+        </material>
+        <material name="green">
+            <color rgba="0 1 0 1"/>
         </material>
         <xacro:macro name="box_inertia" params="m x y z o_xyz o_rpy">

File: src/my_robot_description/urdf/mobile_base.xacro (robot description, xacro)
@@ -13,5 +13,5 @@
                 </geometry>
                 <origin xyz="0 0 ${base_height / 2.0}" rpy="0 0 0" />
-                <material name="blue" />
+                <material name="grey" />
             </visual>
             <collision>

File: src/my_robot_description/urdf/my_robot.urdf.xacro (robot description, xacro)
@@ -4,4 +4,6 @@
     <xacro:include filename="mobile_base.xacro" />
     <xacro:include filename="mobile_base_gazebo.xacro" />
+    <xacro:include filename="water_tank.xacro"/>
+    <xacro:include filename="soap_tank.xacro"/>
     <xacro:include filename="camera.xacro" />
 </robot>
