Commit message: changes regarding the robotic arm

File: src/car_washing_robot_description/urdf/car_washing_robot.urdf.xacro (robot description, xacro)
@@ -7,9 +7,18 @@
     <xacro:include filename="soap_tank.xacro"/>
     <xacro:include filename="camera.xacro" />
-    <xacro:include filename="six_dof_arm.xacro"/>
-    <joint name="base_arm_base_joint" type="fixed">
-        <parent link="base_link"/>
-        <child link="arm_base_link"/>
-        <origin xyz="0 ${base_width/3.0} ${(base_height/2.0)+ 0.08}" rpy="0 0 0"/>
+    <xacro:include filename="test_arm.xacro"/>
+    <xacro:include filename="test_arm_gazebo.xacro"/>
+    <!-- <xacro:include filename="arm_gazebo.xacro"/> -->
+            <!-- Connection Joint Between Mobile Base and Arm -->
+    <!-- <joint name="mobile_base_arm_joint" type="fixed">
+        <parent link="base_link" />
+        <child link="arm_base_link" />
+        <origin xyz="${base_length / 5.0} 0 ${base_height}" rpy="0 0 0" />
+    </joint> -->
+    <!--Connection test2-->
+    <joint name="mobile_base_arm_joint" type="fixed">
+        <parent link="base_link" />
+        <child link="arm_base_link" />
+        <origin xyz="${base_length / 5.0} 0 ${base_height + arm_base_height/2.0}" rpy="0 0 0" />
     </joint>
 </robot>

File: src/car_washing_robot_description/urdf/mobile_base.xacro (robot description, xacro)
@@ -3,5 +3,5 @@
         <xacro:property name="base_length" value="1"/>
         <xacro:property name="base_width" value="0.8"/>
-        <xacro:property name="base_height" value="0.3"/>
+        <xacro:property name="base_height" value="0.26"/>
         <xacro:property name="wheel_radius" value="0.3"/>
         <xacro:property name="wheel_length" value="0.15"/>

Commit message: Removed files and cleaned the workspace

File: src/car_washing_robot_description/urdf/car_washing_robot.urdf.xacro (robot description, xacro)
@@ -7,14 +7,7 @@
     <xacro:include filename="soap_tank.xacro"/>
     <xacro:include filename="camera.xacro" />
-    <xacro:include filename="test_arm.xacro"/>
-    <xacro:include filename="test_arm_gazebo.xacro"/>
-    <!-- <xacro:include filename="arm_gazebo.xacro"/> -->
-            <!-- Connection Joint Between Mobile Base and Arm -->
-    <!-- <joint name="mobile_base_arm_joint" type="fixed">
-        <parent link="base_link" />
-        <child link="arm_base_link" />
-        <origin xyz="${base_length / 5.0} 0 ${base_height}" rpy="0 0 0" />
-    </joint> -->
-    <!--Connection test2-->
+    <xacro:include filename="six_dof_arm.xacro"/>
+    <xacro:include filename="six_dof_arm_gazebo.xacro"/>
+    <!-- Connection Joint Between Mobile Base and Arm -->
     <joint name="mobile_base_arm_joint" type="fixed">
         <parent link="base_link" />

File: src/car_washing_robot_description/urdf/common_properties.xacro (robot description, xacro)
@@ -15,4 +15,7 @@
         <material name="green">
             <color rgba="0 1 0 1"/>
+        </material>
+        <material name="red">
+            <color rgba="1 0 0 1"/>
         </material>
         <xacro:macro name="box_inertia" params="m x y z o_xyz o_rpy">

File: src/car_washing_robot_description/urdf/six_dof_arm.xacro (robot description, xacro)
@@ -1,381 +1,110 @@
-<?xml version="1.0" encoding="utf-8"?>
+<?xml version="1.0"?>
 <robot xmlns:xacro="http://www.ros.org/wiki/xacro">
-  <link
-    name="arm_base_link">
-    <inertial>
-      <origin
-        xyz="0.150569577094829 -0.282065557059584 0.0858444903709998"
-        rpy="0 0 0" />
-      <mass
-        value="3.82869416281393" />
-      <inertia
-        ixx="0.0231805999397633"
-        ixy="-9.35626509492742E-07"
-        ixz="0.000718143477106582"
-        iyy="0.023829421434195"
-        iyz="6.20025735268592E-07"
-        izz="0.0401642921599346" />
-    </inertial>
+<!--Arm base link-->
+    <xacro:property name="arm_base_length" value="0.6" />
+    <xacro:property name="arm_base_width" value="0.8" />
+    <xacro:property name="arm_base_height" value="0.26" />
+    <link name="arm_base_link">
+        <visual>
+            <geometry>
+                <box size="${arm_base_length} ${arm_base_width} ${arm_base_height}" />
+            </geometry>
+            <origin xyz="0 0 0" rpy="0 0 0" />
+            <material name="orange" />
+        </visual>
+        <collision>
+            <geometry>
+                <box size="${arm_base_length} ${arm_base_width} ${arm_base_height}" />
+            </geometry>
+            <origin xyz="0 0 0" rpy="0 0 0" />
+        </collision>
+        <xacro:box_inertia m="0.5" x="${arm_base_length}" y="${arm_base_width}" z="${arm_base_height}"
+                           o_xyz="0 0 0" o_rpy="0 0 0" />
+    </link>
+  <!-- Links and Joints -->
+  <xacro:macro name="arm_link" params="link_name parent_name xyz rpy length radius mass ixx iyy izz">
+    <link name="${link_name}">
+      <visual>
+        <geometry>
+          <cylinder length="${length}" radius="${radius}"/>
+        </geometry>
+        <origin xyz="0 0 ${length/2}" rpy="0 0 0"/>
+        <material name="red"/>
+      </visual>
+      <collision>
+        <geometry>
+          <cylinder length="${length}" radius="${radius}"/>
+        </geometry>
+        <origin xyz="0 0 ${length/2}" rpy="0 0 0"/>
+      </collision>
+      <xacro:cylinder_inertia m="0.3" r="${radius}" l="${length}"
+                                o_xyz="0 0 ${length / 2.0}" o_rpy="0 0 0" />
+    </link>
+    <joint name="${link_name}_joint" type="revolute">
+      <parent link="${parent_name}"/>
+      <child link="${link_name}"/>
+      <origin xyz="${xyz}" rpy="${rpy}"/>
+      <axis xyz="0 1 0"/>
+      <limit lower="${-pi/2}" upper="${pi/2}" effort="100" velocity="100" />
+      <dynamics friction="1.0" damping="5.0" />
+    </joint>
+  </xacro:macro>
+     <!-- Z-axis Rotating Link and Joint -->
+  <xacro:macro name="z_axis_arm_link" params="link_name parent_name xyz rpy length radius mass ixx iyy izz">
+    <link name="${link_name}">
+      <visual>
+        <geometry>
+          <cylinder length="${length}" radius="${radius}"/>
+        </geometry>
+        <origin xyz="0 0 ${length/2}" rpy="0 0 0"/>
+        <material name="blue"/>
+      </visual>
+      <collision>
+        <geometry>
+          <cylinder length="${length}" radius="${radius}"/>
+        </geometry>
+        <origin xyz="0 0 ${length/2}" rpy="0 0 0"/>
+      </collision>
+      <xacro:cylinder_inertia m="0.3" r="${radius}" l="${length}"
+                                o_xyz="0 0 ${length / 2.0}" o_rpy="0 0 0" />
+    </link>
+    <joint name="${link_name}_joint" type="revolute">
+      <parent link="${parent_name}"/>
+      <child link="${link_name}"/>
+      <origin xyz="${xyz}" rpy="${rpy}"/>
+      <axis xyz="0 0 1"/>
+      <limit lower="${-pi/2}" upper="${pi/2}" effort="100" velocity="100" />
+      <dynamics friction="1.0" damping="5.0" />
+    </joint>
+  </xacro:macro>
+  <!-- Instantiate 6 links -->
+  <xacro:z_axis_arm_link link_name="link_1" parent_name="arm_base_link" xyz="${arm_base_width/4.0} 0 0.13" rpy="0 0 0" length="0.2" radius="0.06" mass="1.0" ixx="0.005" iyy="0.005" izz="0.005"/>
+  <xacro:arm_link link_name="link_2" parent_name="link_1" xyz="0 0 0.2" rpy="0 0 0" length="0.2" radius="0.05" mass="0.8" ixx="0.003" iyy="0.003" izz="0.003"/>
+  <xacro:arm_link link_name="link_3" parent_name="link_2" xyz="0 0 0.2" rpy="0 0 0" length="0.15" radius="0.04" mass="0.6" ixx="0.002" iyy="0.002" izz="0.002"/>
+  <xacro:z_axis_arm_link link_name="link_4" parent_name="link_3" xyz="0 0 0.15" rpy="0 0 0" length="0.15" radius="0.04" mass="0.5" ixx="0.0015" iyy="0.0015" izz="0.0015"/>
+  <xacro:arm_link link_name="link_5" parent_name="link_4" xyz="0 0 0.15" rpy="0 0 0" length="0.1" radius="0.03" mass="0.3" ixx="0.001" iyy="0.001" izz="0.001"/>
+  <xacro:arm_link link_name="link_6" parent_name="link_5" xyz="0 0 0.1" rpy="0 0 0" length="0.1" radius="0.03" mass="0.2" ixx="0.0008" iyy="0.0008" izz="0.0008"/>
+    <!-- Camera at the end
+  <link name="camera_link">
     <visual>
-      <origin
-        xyz="0 0 0"
-        rpy="0 0 0" />
       <geometry>
-        <mesh
-          filename="package://car_washing_robot_description/meshes/arm_base_link.STL" />
+        <box size="0.05 0.05 0.05"/>
       </geometry>
-      <material
-        name="">
-        <color
-          rgba="0.247058823529412 0.23921568627451 0.235294117647059 1" />
-      </material>
+      <origin xyz="0 0 0" rpy="0 0 0"/>
+      <material name="grey"/>
     </visual>
     <collision>
-      <origin
-        xyz="0 0 0"
-        rpy="0 0 0" />
       <geometry>
-        <mesh
-          filename="package://car_washing_robot_description/meshes/arm_base_link.STL" />
+        <box size="0.05 0.05 0.05"/>
       </geometry>
+      <origin xyz="0 0 0" rpy="0 0 0"/>
     </collision>
+    <xacro:box_inertia m="0.1" x="0.05" y="0.05" z="0.05"
+                          o_xyz="0 0 0" o_rpy="0 0 0"/>
   </link>
-  <link
-    name="link_1">
-    <inertial>
-      <origin
-        xyz="4.32383283317378E-05 0.0680624071651353 6.52562397435164E-06"
-        rpy="0 0 0" />
-      <mass
-        value="0.496365683666781" />
-      <inertia
-        ixx="0.000792847522971884"
-        ixy="-3.73013993388821E-07"
-        ixz="1.80968680807939E-05"
-        iyy="0.000184926812457533"
-        iyz="-4.97697758356282E-09"
-        izz="0.000717881898216823" />
-    </inertial>
-    <visual>
-      <origin
-        xyz="0 0 0"
-        rpy="0 0 0" />
-      <geometry>
-        <mesh
-          filename="package://car_washing_robot_description/meshes/link_1.STL" />
-      </geometry>
-      <material
-        name="">
-        <color
-          rgba="0.898039215686275 0.917647058823529 0.929411764705882 1" />
-      </material>
-    </visual>
-    <collision>
-      <origin
-        xyz="0 0 0"
-        rpy="0 0 0" />
-      <geometry>
-        <mesh
-          filename="package://car_washing_robot_description/meshes/link_1.STL" />
-      </geometry>
-    </collision>
-  </link>
-  <joint
-    name="joint_1"
-    type="continuous">
-    <origin
-      xyz="0.15423 -0.28206 0.10149"
-      rpy="1.5708 0 0.43749" />
-    <parent
-      link="arm_base_link" />
-    <child
-      link="link_1" />
-    <axis
-      xyz="0 1 0" />
-  </joint>
-  <link
-    name="link_2">
-    <inertial>
-      <origin
-        xyz="0.0338354479920845 -0.0064322169652048 -0.00245407284264082"
-        rpy="0 0 0" />
-      <mass
-        value="0.252006469213197" />
-      <inertia
-        ixx="6.24106980967512E-05"
-        ixy="2.122889857404E-05"
-        ixz="8.94621229356148E-06"
-        iyy="0.000169543347753182"
-        iyz="-3.84314642165744E-07"
-        izz="0.000182079065869168" />
-    </inertial>
-    <visual>
-      <origin
-        xyz="0 0 0"
-        rpy="0 0 0" />
-      <geometry>
-        <mesh
-          filename="package://car_washing_robot_description/meshes/link_2.STL" />
-      </geometry>
-      <material
-        name="">
-        <color
-          rgba="0.898039215686275 0.917647058823529 0.929411764705882 1" />
-      </material>
-    </visual>
-    <collision>
-      <origin
-        xyz="0 0 0"
-        rpy="0 0 0" />
-      <geometry>
-        <mesh
-          filename="package://car_washing_robot_description/meshes/link_2.STL" />
-      </geometry>
-    </collision>
-  </link>
-  <joint
-    name="joint_2"
-    type="revolute">
-    <origin
-      xyz="0 0.112 0"
-      rpy="1.5708 0 2.4755" />
-    <parent
-      link="link_1" />
-    <child
-      link="link_2" />
-    <axis
-      xyz="0 1 0" />
-    <limit
-      lower="-1.57"
-      upper="1.57"
-      effort="10"
-      velocity="1.57" />
-  </joint>
-  <link
-    name="link_3">
-    <inertial>
-      <origin
-        xyz="-0.0270205188287359 -0.00383049369840976 -0.0142531927255568"
-        rpy="0 0 0" />
-      <mass
-        value="0.343635149193939" />
-      <inertia
-        ixx="0.00028538664881932"
-        ixy="-9.66773270784163E-06"
-        ixz="-4.92482264612374E-06"
-        iyy="0.000529175475076648"
-        iyz="4.3261957062028E-05"
-        izz="0.000338633695459992" />
-    </inertial>
-    <visual>
-      <origin
-        xyz="0 0 0"
-        rpy="0 0 0" />
-      <geometry>
-        <mesh
-          filename="package://car_washing_robot_description/meshes/link_3.STL" />
-      </geometry>
-      <material
-        name="">
-        <color
-          rgba="0.898039215686275 0.917647058823529 0.929411764705882 1" />
-      </material>
-    </visual>
-    <collision>
-      <origin
-        xyz="0 0 0"
-        rpy="0 0 0" />
-      <geometry>
-        <mesh
-          filename="package://car_washing_robot_description/meshes/link_3.STL" />
-      </geometry>
-    </collision>
-  </link>
-  <joint
-    name="joint_3"
-    type="revolute">
-    <origin
-      xyz="0.065 0 0"
-      rpy="1.5708 0.62232 3.1416" />
-    <parent
-      link="link_2" />
-    <child
-      link="link_3" />
-    <axis
-      xyz="0 0 1" />
-    <limit
-      lower="-1.57"
-      upper="1.57"
-      effort="10"
-      velocity="1.57" />
-  </joint>
-  <link
-    name="link_4">
-    <inertial>
-      <origin
-        xyz="0.00315043687013407 0.00823334083490718 -0.0153088125607234"
-        rpy="0 0 0" />
-      <mass
-        value="0.458108386971292" />
-      <inertia
-        ixx="0.000266524923789775"
-        ixy="-4.83010597650581E-05"
-        ixz="-2.58452901540373E-05"
-        iyy="0.000231242852741601"
-        iyz="-7.692645775569E-06"
-        izz="0.000378867067607329" />
-    </inertial>
-    <visual>
-      <origin
-        xyz="0 0 0"
-        rpy="0 0 0" />
-      <geometry>
-        <mesh
-          filename="package://car_washing_robot_description/meshes/link_4.STL" />
-      </geometry>
-      <material
-        name="">
-        <color
-          rgba="0.898039215686275 0.917647058823529 0.929411764705882 1" />
-      </material>
-    </visual>
-    <collision>
-      <origin
-        xyz="0 0 0"
-        rpy="0 0 0" />
-      <geometry>
-        <mesh
-          filename="package://car_washing_robot_description/meshes/link_4.STL" />
-      </geometry>
-    </collision>
-  </link>
-  <joint
-    name="joint_4"
-    type="revolute">
-    <origin
-      xyz="-0.0652500000000006 0 0"
-      rpy="0 0 1.38288301124323" />
-    <parent
-      link="link_3" />
-    <child
-      link="link_4" />
-    <axis
-      xyz="0 0 1" />
-    <limit
-      lower="-1.57"
-      upper="1.57"
-      effort="10"
-      velocity="1.57" />
-  </joint>
-  <link
-    name="link_5">
-    <inertial>
-      <origin
-        xyz="0.00289484913778473 0.00414654326045577 0.0215505654647544"
-        rpy="0 0 0" />
-      <mass
-        value="0.126917113445138" />
-      <inertia
-        ixx="5.56063236989531E-05"
-        ixy="-1.6838052978347E-06"
-        ixz="-1.46179701383522E-06"
-        iyy="3.36435019532127E-05"
-        iyz="-2.18123980266177E-06"
-        izz="4.54057563337419E-05" />
-    </inertial>
-    <visual>
-      <origin
-        xyz="0 0 0"
-        rpy="0 0 0" />
-      <geometry>
-        <mesh
-          filename="package://car_washing_robot_description/meshes/link_5.STL" />
-      </geometry>
-      <material
-        name="">
-        <color
-          rgba="0.898039215686275 0.917647058823529 0.929411764705882 1" />
-      </material>
-    </visual>
-    <collision>
-      <origin
-        xyz="0 0 0"
-        rpy="0 0 0" />
-      <geometry>
-        <mesh
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