Commit message: Increased mass of base to avoid flipping & increased friction and damping to avoid arm movement due to gravity

File: src/car_washing_robot_description/urdf/mobile_base.xacro (robot description, xacro)
@@ -21,5 +21,5 @@
                 <origin xyz="0 0 ${base_height / 2.0}" rpy="0 0 0" />
             </collision>
-            <xacro:box_inertia m="5.0" x="${base_length}" y="${base_width}" z="${base_height}"
+            <xacro:box_inertia m="40.0" x="${base_length}" y="${base_width}" z="${base_height}"
                                o_xyz="0 0 ${base_height / 2.0}" o_rpy="0 0 0"/>
         </link>

File: src/car_washing_robot_description/urdf/six_dof_arm.xacro (robot description, xacro)
@@ -47,5 +47,5 @@
       <axis xyz="0 1 0"/>
       <limit lower="${-pi/2}" upper="${pi/2}" effort="100" velocity="100" />
-      <dynamics friction="1.0" damping="5.0" />
+      <dynamics friction="10.0" damping="50.0" />
     </joint>
   </xacro:macro>
@@ -75,5 +75,5 @@
       <axis xyz="0 0 1"/>
       <limit lower="${-pi/2}" upper="${pi/2}" effort="100" velocity="100" />
-      <dynamics friction="1.0" damping="5.0" />
+      <dynamics friction="10.0" damping="50.0" />
     </joint>
   </xacro:macro>
