Commit message: lidar

File: src/car_washing_robot_description/urdf/lidar.xacro (robot description, xacro)
@@ -25,18 +25,41 @@
     </joint>
     <gazebo reference="base_scan">
-        <sensor name="lidar" type="gpu_lidar">
+        <sensor name="laser" type="gpu_lidar">
+            <pose> 0 0 0 0 0 0 </pose>
+            <always_on>true</always_on>
+            <visualize>true</visualize>
             <update_rate>10</update_rate>
-            <topic>scan</topic>
-            <frame_name>base_scan</frame_name>
+            <!-- <topic>model/car_washing_robot/scan</topic> -->
+            <!-- <topic>scan</topic> -->
+            <gz_frame_id>base_scan</gz_frame_id>
             <lidar>
-                <horizontal>
-                    <samples>180</samples>
-                    <min_angle>-1.5708</min_angle>
-                    <max_angle>1.5708</max_angle>
-                </horizontal>
+                <scan>
+                    <horizontal>
+                    <samples>720</samples>
+                    <resolution>1</resolution>
+                    <min_angle>-3.14</min_angle>
+                    <max_angle>3.14</max_angle>
+                    </horizontal>
+                </scan>
                 <range>
-                    <min>0.12</min>
+                    <min>0.05</min>
                     <max>10.0</max>
+                    <resolution>0.01</resolution>
                 </range>
+                <noise>
+                    <type>gaussian</type>
+                    <mean>0.0</mean>
+                    <stddev>0.01</stddev>
+                </noise>
+                <!-- <ignore>
+                    <link>arm_base_link</link>
+                    <link>robot_arm_link_1</link>
+                    <link>robot_arm_link_2</link>
+                    <link>robot_arm_link_3</link>
+                    <link>robot_arm_link_4</link>
+                    <link>robot_arm_link_5</link>
+                    <link>robot_arm_link_6</link>
+                    <link>soap_tank</link>
+                </ignore> -->
             </lidar>
         </sensor>

Commit message: Lidar changes

File: src/car_washing_robot_description/urdf/lidar.xacro (robot description, xacro)
@@ -3,5 +3,5 @@
     <xacro:property name="base_scan_radius" value="0.05"/>
     <xacro:property name="base_scan_length" value="0.05"/>
-    <link name="base_scan">
+    <link name="base_scan_link">
         <visual>
             <geometry>
@@ -20,17 +20,19 @@
     </link>
     <joint name="base_scan_joint" type="fixed">
-        <parent link="base_link"/>
-        <child link="base_scan"/>
-        <origin xyz="${arm_base_width/2.0} 0 ${arm_base_height + base_height}" rpy="0 0 0"/>
+        <parent link="arm_base_link"/>
+        <!-- <parent link="base_link"/> -->
+        <child link="base_scan_link"/>
+        <origin xyz="${arm_base_width/4.0} 0 ${arm_base_height/2.0}" rpy="0 0 0"/>
     </joint>
-    <gazebo reference="base_scan">
-        <sensor name="laser" type="gpu_lidar">
+    <gazebo reference="base_scan_link">
+        <sensor name="base_scan_sensor" type="gpu_lidar">
             <pose> 0 0 0 0 0 0 </pose>
             <always_on>true</always_on>
             <visualize>true</visualize>
             <update_rate>10</update_rate>
-            <!-- <topic>model/car_washing_robot/scan</topic> -->
-            <!-- <topic>scan</topic> -->
-            <gz_frame_id>base_scan</gz_frame_id>
+            <topic>model/car_washing_robot/scan</topic>
+            <!-- <topic>/scan</topic> -->
+            <!-- <frame_id>base_scan_link</frame_id> -->
+            <frame>base_scan_link</frame>
             <lidar>
                 <scan>
@@ -38,6 +40,6 @@
                     <samples>720</samples>
                     <resolution>1</resolution>
-                    <min_angle>-3.14</min_angle>
-                    <max_angle>3.14</max_angle>
+                    <min_angle>-2.30</min_angle> <!-- -131.78 degrees-->
+                    <max_angle>2.30</max_angle>  <!--  131.78 degrees-->
                     </horizontal>
                 </scan>
@@ -52,14 +54,4 @@
                     <stddev>0.01</stddev>
                 </noise>
-                <!-- <ignore>
-                    <link>arm_base_link</link>
-                    <link>robot_arm_link_1</link>
-                    <link>robot_arm_link_2</link>
-                    <link>robot_arm_link_3</link>
-                    <link>robot_arm_link_4</link>
-                    <link>robot_arm_link_5</link>
-                    <link>robot_arm_link_6</link>
-                    <link>soap_tank</link>
-                </ignore> -->
             </lidar>
         </sensor>

File: src/car_washing_robot_description/urdf/mobile_base_gazebo.xacro (robot description, xacro)
@@ -14,5 +14,5 @@
             <right_joint>base_right_wheel_joint</right_joint>
             <wheel_separation>0.45</wheel_separation>
-            <wheel_radius>0.1</wheel_radius>
+            <wheel_radius>0.3</wheel_radius>
             <frame_id>odom</frame_id>
             <child_frame_id>base_footprint</child_frame_id>
@@ -28,3 +28,18 @@
         </plugin>
     </gazebo>
+    <!-- <gazebo>
+        <plugin
+            filename="gz-sim-pose-publisher-system"
+            name="gz::sim::systems::PosePublisher">
+            <publish_link_pose>true</publish_link_pose>
+            <publish_sensor_pose>true</publish_sensor_pose>
+            <publish_collision_pose>false</publish_collision_pose>
+            <publish_visual_pose>false</publish_visual_pose>
+            <publish_nested_model_pose>false</publish_nested_model_pose>
+            <use_pose_vector_msg>true</use_pose_vector_msg>
+            <static_publisher>false</static_publisher>
+            <static_update_frequency>100</static_update_frequency>
+            <update_frequency>100</update_frequency>
+        </plugin>
+    </gazebo> -->
 </robot>
